Commit message: Rename package and fix gazebo bridge bug

File: src/almu_rover/urdf/basic_rover.urdf.xacro (robot description, xacro)
@@ -1,9 +1,12 @@
 <?xml version="1.0"?>
-<robot name="almu_rover">
-    <link name="base_link">
+<robot name="almu_rover" xmlns:xacro="http://www.ros.org/wiki/xacro">
+    <xacro:include filename="$(find almu_rover)/urdf/materials.urdf.xacro" />
+    <link name="base_link" />
+    <link name="body">
         <visual>
             <geometry>
                 <box size="1.2 1.0 0.3"/>
             </geometry>
+            <!-- <material name="blue" /> -->
             <material name="LightGrey">
                 <color rgba="0.7 0.7 0.7 1.0"/>
@@ -21,4 +24,10 @@
         </inertial>
     </link>
+    <joint name="body_joint" type="fixed">
+        <parent link="base_link"/>
+        <child link="body"/>
+        <origin xyz="0 0 0" rpy="0 0 0"/>
+        <axis xyz="0 0 0"/>
+    </joint>
     <link name="front_left_arm">
         <visual>
@@ -43,5 +52,5 @@
     </link>
     <joint name="front_left_joint" type="fixed">
-        <parent link="base_link"/>
+        <parent link="body"/>
         <child link="front_left_arm"/>
         <origin xyz="0.5 0.6 0" rpy="0 ${pi / 2} 0"/>
@@ -70,5 +79,5 @@
     </link>
     <joint name="front_right_joint" type="fixed">
-        <parent link="base_link"/>
+        <parent link="body"/>
         <child link="front_right_arm"/>
         <origin xyz="0.5 -0.6 0" rpy="0 ${pi / 2} 0"/>
@@ -98,5 +107,5 @@
     </link>
     <joint name="rear_left_joint" type="fixed">
-        <parent link="base_link"/>
+        <parent link="body"/>
         <child link="rear_left_arm"/>
         <origin xyz="-0.5 0.6 0" rpy="0 ${pi / 2} 0"/>
@@ -126,5 +135,5 @@
     </link>
     <joint name="rear_right_joint" type="fixed">
-        <parent link="base_link"/>
+        <parent link="body"/>
         <child link="rear_right_arm"/>
         <origin xyz="-0.5 -0.6 0" rpy="0 ${pi / 2} 0"/>
