Commit message: Add front camera

File: src/maly_woz_description/urdf/basic_rover.urdf.xacro (robot description, xacro)
@@ -37,4 +37,48 @@
   <xacro:leg suffix="rear_right" parent="body" front="-1" left="-1"
              x_offset="-0.5" y_offset="-0.5" z_offset="0.0" />
+  <!-- TODO extract camera to macro -->
+  <link name="camera_front">
+    <inertial>
+      <mass value="0.3"/>
+      <origin xyz="0 0 0" rpy="0 0 0"/>
+      <xacro:solid_cuboid_inertia m="0.1" w="0.1" d="0.1" h="0.1" />
+    </inertial>
+    <collision>
+      <geometry>
+        <box size="0.1 0.1 0.1"/>
+      </geometry>
+    </collision>
+    <visual>
+      <geometry>
+        <box size="0.1 0.1 0.1"/>
+      </geometry>
+      <material name="black" />
+    </visual>
+  </link>
+  <gazebo reference="camera_front">
+    <sensor name="camera_front" type="camera">
+      <camera>
+        <horizontal_fov>1.047</horizontal_fov>
+        <image>
+          <width>320</width>
+          <height>240</height>
+        </image>
+        <clip>
+          <near>0.1</near>
+          <far>100</far>
+        </clip>
+      </camera>
+      <always_on>1</always_on>
+      <update_rate>30</update_rate>
+      <visualize>true</visualize>
+      <topic>camera_front/image_raw</topic>
+    </sensor>
+  </gazebo>
+  <joint name="camera_front_joint" type="fixed">
+    <parent link="body"/>
+    <child link="camera_front"/>
+    <origin xyz="0.5 0 0.3" rpy="0 0 0"/>
+    <axis xyz="0 0 0"/>
+  </joint>
   <gazebo>
     <plugin

Commit message: Add depth camera

File: src/maly_woz_description/urdf/basic_rover.urdf.xacro (robot description, xacro)
@@ -57,10 +57,16 @@
   </link>
   <gazebo reference="camera_front">
+    <!-- D435 depth camera -->
     <sensor name="camera_front" type="camera">
-      <camera>
-        <horizontal_fov>1.047</horizontal_fov>
+      <always_on>1</always_on>
+      <update_rate>30</update_rate>
+      <visualize>1</visualize>
+      <topic>camera_front/image_raw</topic>
+      <camera name="d435">
+        <horizontal_fov>1.21126</horizontal_fov>
         <image>
-          <width>320</width>
-          <height>240</height>
+          <width>640</width>
+          <height>480</height>
+          <format>RGB_INT8</format>
         </image>
         <clip>
@@ -68,9 +74,32 @@
           <far>100</far>
         </clip>
+        <noise>
+          <type>gaussian</type>
+          <mean>0</mean>
+          <stddev>0.007</stddev>
+        </noise>
       </camera>
+    </sensor>
+    <sensor name="depth_front" type="depth_camera">
       <always_on>1</always_on>
       <update_rate>30</update_rate>
-      <visualize>true</visualize>
-      <topic>camera_front/image_raw</topic>
+      <visualize>0</visualize>
+      <topic>depth_front/depth</topic>
+      <camera name="d435_depth">
+        <horizontal_fov>1.48702</horizontal_fov>
+        <image>
+          <width>1280</width>
+          <height>720</height>
+        </image>
+        <clip>
+          <near>0.1</near>
+          <far>10</far>
+        </clip>
+        <noise>
+          <type>gaussian</type>
+          <mean>0</mean>
+          <stddev>0.1</stddev>
+        </noise>
+      </camera>
     </sensor>
   </gazebo>

File: src/maly_woz_description/urdf/leg.urdf.xacro (robot description, xacro)
@@ -42,5 +42,5 @@
           <cylinder radius="0.1" length="0.1"/>
         </geometry>
-        <origin xyz="0 0 0.05" rpy="0 0 0"/>
+        <origin xyz="0 0 ${left * 0.05}" rpy="0 0 0"/>
       </collision>
       <inertial>

Commit message: Use more reasonable values for the rover

File: src/maly_woz_description/urdf/basic_rover.urdf.xacro (robot description, xacro)
@@ -4,9 +4,13 @@
   <xacro:include filename="$(find maly_woz_description)/urdf/materials.urdf.xacro" />
   <xacro:include filename="$(find maly_woz_description)/urdf/inertia.urdf.xacro" />
+  <xacro:property name="wheel_radius" value="0.1"/>
+  <xacro:property name="leg_length" value="0.2"/>
+  <xacro:property name="chassis_length" value="0.8"/>
+  <xacro:property name="chassis_width" value="0.5"/>
   <link name="base_link" />
   <link name="body">
     <visual>
       <geometry>
-        <box size="1.2 1.0 0.3"/>
+        <box size="${chassis_length} ${chassis_width} 0.3"/>
       </geometry>
       <material name="blue" />
@@ -14,11 +18,11 @@
     <collision>
       <geometry>
-        <box size="1.2 1.0 0.3"/>
+        <box size="${chassis_length} ${chassis_width} 0.3"/>
       </geometry>
     </collision>
     <inertial>
-      <mass value="1.0"/>
+      <mass value="3.0"/>
       <origin xyz="0 0 0" rpy="0 0 0"/>
-      <inertia ixx="0.0001" ixy="0.0" ixz="0.0" iyy="0.0001" iyz="0.0" izz="0.0001"/>
+      <xacro:solid_cuboid_inertia m="3.0" w="${chassis_width}" d="${chassis_length}" h="0.3" />
     </inertial>
   </link>
@@ -26,19 +30,23 @@
     <parent link="base_link"/>
     <child link="body"/>
-    <origin xyz="0 0 0" rpy="0 0 0"/>
+    <origin xyz="0 0 ${wheel_radius + leg_length}" rpy="0 0 0"/>
     <axis xyz="0 0 0"/>
   </joint>
   <xacro:leg suffix="front_left" parent="body" front="1" left="1"
-             x_offset="0.5" y_offset="0.5" z_offset="0.0" />
+             x_offset="${chassis_length / 2}" y_offset="${chassis_width / 2}" z_offset="0.0"
+             wheel_radius="${wheel_radius}" leg_length="${leg_length}" />
   <xacro:leg suffix="front_right" parent="body" front="1" left="-1"
-             x_offset="0.5" y_offset="-0.5" z_offset="0.0" />
+             x_offset="${chassis_length / 2}" y_offset="-${chassis_width / 2}" z_offset="0.0"
+             wheel_radius="${wheel_radius}" leg_length="${leg_length}" />
   <xacro:leg suffix="rear_left" parent="body" front="-1" left="1"
-             x_offset="-0.5" y_offset="0.5" z_offset="0.0" />
+             x_offset="-${chassis_length / 2}" y_offset="${chassis_width / 2}" z_offset="0.0"
+             wheel_radius="${wheel_radius}" leg_length="${leg_length}" />
   <xacro:leg suffix="rear_right" parent="body" front="-1" left="-1"
-             x_offset="-0.5" y_offset="-0.5" z_offset="0.0" />
+             x_offset="-${chassis_length / 2}" y_offset="-${chassis_width / 2}" z_offset="0.0"
+             wheel_radius="${wheel_radius}" leg_length="${leg_length}" />
   <!-- TODO extract camera to macro -->
   <link name="camera_front">
     <inertial>
-      <mass value="0.3"/>
+      <mass value="0.1"/>
       <origin xyz="0 0 0" rpy="0 0 0"/>
       <xacro:solid_cuboid_inertia m="0.1" w="0.1" d="0.1" h="0.1" />
@@ -107,5 +115,5 @@
     <parent link="body"/>
     <child link="camera_front"/>
-    <origin xyz="0.5 0 0.3" rpy="0 0 0"/>
+    <origin xyz="0.4 0 0.2" rpy="0 ${20 * pi / 180} 0"/>
     <axis xyz="0 0 0"/>
   </joint>
@@ -119,5 +127,5 @@
       <right_joint>wheel_rear_right_joint</right_joint>
       <wheel_separation>${1.0 + 2 * 0.05 + 0.05}</wheel_separation>
-      <wheel_radius>0.1</wheel_radius>
+      <wheel_radius>${wheel_radius}</wheel_radius>
       <odom_publish_frequency>30</odom_publish_frequency>
       <max_linear_acceleration>5</max_linear_acceleration>

File: src/maly_woz_description/urdf/leg.urdf.xacro (robot description, xacro)
@@ -1,22 +1,24 @@
 <?xml version="1.0"?>
 <robot xmlns:xacro="http://www.ros.org/wiki/xacro">
-  <xacro:macro name="leg" params="suffix parent front left x_offset y_offset z_offset">
+  <xacro:macro name="leg" params="suffix parent front left x_offset y_offset z_offset
+                                  wheel_radius leg_length">
     <link name="leg_${suffix}">
       <visual>
         <geometry>
-          <box size="0.5 0.1 0.1"/>
+          <box size="${leg_length} 0.1 0.1"/>
         </geometry>
         <material name="blue" />
-        <origin xyz="0.25 0 0" rpy="0 0 0"/>
+        <origin xyz="${leg_length / 2} 0 0" rpy="0 0 0"/>
       </visual>
       <collision>
         <geometry>
-          <box size="0.5 0.2 0.2"/>
+          <box size="${leg_length} 0.2 0.2"/>
         </geometry>
+        <origin xyz="${leg_length / 2} 0 0" rpy="0 0 0"/>
       </collision>
       <inertial>
         <mass value="0.3"/>
-        <origin xyz="0 0 0" rpy="0 0 0"/>
-        <xacro:solid_cuboid_inertia m="0.3" w="0.5" d="0.2" h="0.2" />
+        <origin xyz="${leg_length / 2} 0 0" rpy="0 0 0"/>
+        <xacro:solid_cuboid_inertia m="0.3" w="${leg_length}" d="0.2" h="0.2" />
       </inertial>
     </link>
@@ -26,5 +28,5 @@
       <origin
         xyz="${x_offset} ${y_offset + left * 0.05} ${z_offset}"
-        rpy="0 ${(pi / 2) - (front * pi * 20 / 180)} 0"
+        rpy="0 ${pi / 2} 0"
       />
       <axis xyz="0 0 1"/>
@@ -33,5 +35,5 @@
       <visual>
         <geometry>
-          <cylinder radius="0.1" length="0.1"/>
+          <cylinder radius="${wheel_radius}" length="0.1"/>
         </geometry>
         <material name="black" />
@@ -40,24 +42,25 @@
       <collision>
         <geometry>
-          <cylinder radius="0.1" length="0.1"/>
+          <cylinder radius="${wheel_radius}" length="0.1"/>
         </geometry>
         <origin xyz="0 0 ${left * 0.05}" rpy="0 0 0"/>
       </collision>
       <inertial>
-        <mass value="0.3"/>
-        <origin xyz="0 0 0" rpy="0 0 0"/>
-        <xacro:solid_cylinder_inertia m="0.1" r="0.1" h="0.1" />
+        <mass value="0.1"/>
+        <xacro:solid_cylinder_inertia m="0.1" r="${wheel_radius}" h="0.1" />
+        <origin xyz="0 0 ${left * 0.05}" rpy="0 0 0"/>
       </inertial>
     </link>
     <gazebo reference="wheel_${suffix}">
       <collision>
+        <pose>0 0 ${left * 0.05} 0 0 0</pose>
         <surface>
           <friction>
             <ode>
-              <mu>1</mu>
+              <mu>1.0</mu>
               <mu2>1</mu2>
-              <slip1>0.5</slip1>
+              <slip1>0</slip1>
               <slip2>0</slip2>
-              <fdir1>0 0 1</fdir1>
+              <fdir1>1 0 0</fdir1>
             </ode>
           </friction>
@@ -68,7 +71,9 @@
       <parent link="leg_${suffix}"/>
       <child link="wheel_${suffix}"/>
-      <origin xyz="0.5 ${left * 0.05} 0" rpy="${-pi / 2} 0 0"/>
+      <origin xyz="${leg_length} ${left * 0.05} 0" rpy="${-pi / 2} 0 0"/>
       <axis xyz="0 0 1"/>
       <limit effort="1000.0" lower="-1e300" upper="1e300" velocity="1e300"/>
+      <dynamics damping="1.0" friction="0.0"/>
+      <joint_properties damping="0.2" friction="0.2"/>
     </joint>
   </xacro:macro>

Commit message: Add proper Intel RealSense D435 sensor

File: src/maly_woz_description/urdf/basic_rover.urdf.xacro (robot description, xacro)
@@ -4,4 +4,5 @@
   <xacro:include filename="$(find maly_woz_description)/urdf/materials.urdf.xacro" />
   <xacro:include filename="$(find maly_woz_description)/urdf/inertia.urdf.xacro" />
+  <xacro:include filename="$(find maly_woz_description)/urdf/sensors/realsense_d435/realsense_d435.urdf.xacro" />
   <xacro:property name="wheel_radius" value="0.1"/>
   <xacro:property name="leg_length" value="0.2"/>
@@ -45,77 +46,7 @@
              x_offset="-${chassis_length / 2}" y_offset="-${chassis_width / 2}" z_offset="0.0"
              wheel_radius="${wheel_radius}" leg_length="${leg_length}" />
-  <!-- TODO extract camera to macro -->
-  <link name="camera_front">
-    <inertial>
-      <mass value="0.1"/>
-      <origin xyz="0 0 0" rpy="0 0 0"/>
-      <xacro:solid_cuboid_inertia m="0.1" w="0.1" d="0.1" h="0.1" />
-    </inertial>
-    <collision>
-      <geometry>
-        <box size="0.1 0.1 0.1"/>
-      </geometry>
-    </collision>
-    <visual>
-      <geometry>
-        <box size="0.1 0.1 0.1"/>
-      </geometry>
-      <material name="black" />
-    </visual>
-  </link>
-  <gazebo reference="camera_front">
-    <!-- D435 depth camera -->
-    <sensor name="camera_front" type="camera">
-      <always_on>1</always_on>
-      <update_rate>30</update_rate>
-      <visualize>1</visualize>
-      <topic>camera_front/image_raw</topic>
-      <camera name="d435">
-        <horizontal_fov>1.21126</horizontal_fov>
-        <image>
-          <width>640</width>
-          <height>480</height>
-          <format>RGB_INT8</format>
-        </image>
-        <clip>
-          <near>0.1</near>
-          <far>100</far>
-        </clip>
-        <noise>
-          <type>gaussian</type>
-          <mean>0</mean>
-          <stddev>0.007</stddev>
-        </noise>
-      </camera>
-    </sensor>
-    <sensor name="depth_front" type="depth_camera">
-      <always_on>1</always_on>
-      <update_rate>30</update_rate>
-      <visualize>0</visualize>
-      <topic>depth_front/depth</topic>
-      <camera name="d435_depth">
-        <horizontal_fov>1.48702</horizontal_fov>
-        <image>
-          <width>1280</width>
-          <height>720</height>
-        </image>
-        <clip>
-          <near>0.1</near>
-          <far>10</far>
-        </clip>
-        <noise>
-          <type>gaussian</type>
-          <mean>0</mean>
-          <stddev>0.1</stddev>
-        </noise>
-      </camera>
-    </sensor>
-  </gazebo>
-  <joint name="camera_front_joint" type="fixed">
-    <parent link="body"/>
-    <child link="camera_front"/>
+  <xacro:realsense_d435 prefix="realsense_front" parent="body">
     <origin xyz="0.4 0 0.2" rpy="0 ${20 * pi / 180} 0"/>
-    <axis xyz="0 0 0"/>
-  </joint>
+  </xacro:realsense_d435>
   <gazebo>
     <plugin
