Commit message: Fix gazebo physics bug

File: src/maly_woz_description/urdf/leg.urdf.xacro (robot description, xacro)
@@ -42,22 +42,4 @@
           <cylinder radius="0.1" length="0.1"/>
         </geometry>
-        <surface>
-          <!-- TODO there is probably some bug with friction, we can't turn really well -->
-          <friction>
-            <ode>
-              <mu>1</mu>
-              <mu2>0.1</mu2>
-              <slip1>0.035</slip1>
-              <slip2>0</slip2>
-              <fdir1>0 0 1</fdir1>
-            </ode>
-            <bullet>
-              <friction>1</friction>
-              <friction2>0.1</friction2>
-              <rolling_friction>0.1</rolling_friction>
-              <spinning_friction>0.1</spinning_friction>
-            </bullet>
-          </friction>
-        </surface>
         <origin xyz="0 0 0.05" rpy="0 0 0"/>
       </collision>
@@ -68,4 +50,19 @@
       </inertial>
     </link>
+    <gazebo reference="wheel_${suffix}">
+      <collision>
+        <surface>
+          <friction>
+            <ode>
+              <mu>1</mu>
+              <mu2>1</mu2>
+              <slip1>0.5</slip1>
+              <slip2>0</slip2>
+              <fdir1>0 0 1</fdir1>
+            </ode>
+          </friction>
+        </surface>
+      </collision>
+    </gazebo>
     <joint name="wheel_${suffix}_joint" type="revolute">
       <parent link="leg_${suffix}"/>

Commit message: Playing with nav and sim parameters

File: src/maly_woz_description/urdf/leg.urdf.xacro (robot description, xacro)
@@ -35,5 +35,6 @@
       <visual>
         <geometry>
-          <cylinder radius="${wheel_radius}" length="0.1"/>
+          <!-- <cylinder radius="${wheel_radius}" length="0.1"/> -->
+          <sphere radius="${wheel_radius}"/>
         </geometry>
         <material name="black" />
@@ -42,5 +43,6 @@
       <collision>
         <geometry>
-          <cylinder radius="${wheel_radius}" length="0.1"/>
+          <!-- <cylinder radius="${wheel_radius}" length="0.1"/> -->
+          <sphere radius="${wheel_radius}"/>
         </geometry>
         <origin xyz="0 0 ${left * 0.05}" rpy="0 0 0"/>
@@ -58,10 +60,20 @@
           <friction>
             <ode>
+              <mu>0.5</mu>
+              <mu2>1.0</mu2>
+              <fdir1>0 0 1</fdir1>
+            </ode>
+            <bullet>
+              <friction>1</friction>
+              <friction2>1</friction2>
+              <rolling_friction>0.1</rolling_friction>
+            </bullet>
+            <!-- <ode>
               <mu>1.0</mu>
-              <mu2>1</mu2>
+              <mu2>0.99</mu2>
               <slip1>0</slip1>
-              <slip2>0</slip2>
+              <slip2>0.01</slip2>
               <fdir1>1 0 0</fdir1>
-            </ode>
+            </ode> -->
           </friction>
         </surface>
@@ -74,6 +86,6 @@
       <axis xyz="0 0 1"/>
       <limit effort="1000.0" lower="-1e300" upper="1e300" velocity="1e300"/>
-      <dynamics damping="1.0" friction="0.0"/>
-      <joint_properties damping="0.2" friction="0.2"/>
+      <dynamics damping="0.0" friction="0.0"/>
+      <joint_properties damping="0.0" friction="0.0"/>
     </joint>
   </xacro:macro>
