Commit message: Add IMU to simulation

File: src/maly_woz_description/urdf/sensors/realsense_d435/realsense_d435.urdf.xacro (robot description, xacro)
@@ -33,4 +33,10 @@
       <child link="${prefix}_optical_frame"/>
       <origin xyz="0.02 0 0" rpy="0 0 0"/>
+    </joint>
+    <link name="${prefix}_imu_frame" />
+    <joint name="${prefix}_imu_joint" type="fixed">
+      <parent link="${prefix}_frame"/>
+      <child link="${prefix}_imu_frame"/>
+      <origin xyz="0 0 0" rpy="0 0 0"/>
     </joint>
     <gazebo reference="${prefix}_optical_frame">
@@ -84,4 +90,13 @@
       </sensor>
     </gazebo>
+    <gazebo reference="${prefix}_imu_frame">
+      <sensor name="imu" type="imu">
+        <gz_frame_id>${prefix}_imu_frame</gz_frame_id>
+        <always_on>1</always_on>
+        <update_rate>100</update_rate>
+        <visualize>true</visualize>
+        <topic>${prefix}/imu</topic>
+      </sensor>
+    </gazebo>
     <joint name="${prefix}_joint" type="fixed">
       <parent link="${parent}"/>

Commit message: Fix bugs with bad projection matrix and rotated optical frame

File: src/maly_woz_description/urdf/sensors/realsense_d435/realsense_d435.urdf.xacro (robot description, xacro)
@@ -28,9 +28,15 @@
       </visual>
     </link>
+    <link name="${prefix}_sensor_frame" />
+    <joint name="${prefix}_sensor_joint" type="fixed">
+      <parent link="${prefix}_frame"/>
+      <child link="${prefix}_sensor_frame"/>
+      <origin xyz="0.02 0 0" rpy="0 0 0"/>
+    </joint>
     <link name="${prefix}_optical_frame" />
     <joint name="${prefix}_optical_joint" type="fixed">
-      <parent link="${prefix}_frame"/>
+      <parent link="${prefix}_sensor_frame"/>
       <child link="${prefix}_optical_frame"/>
-      <origin xyz="0.02 0 0" rpy="0 0 0"/>
+      <origin xyz="0 0 0" rpy="${-pi / 2} 0 ${-pi / 2}"/>
     </joint>
     <link name="${prefix}_imu_frame" />
@@ -40,10 +46,11 @@
       <origin xyz="0 0 0" rpy="0 0 0"/>
     </joint>
-    <gazebo reference="${prefix}_optical_frame">
+    <gazebo reference="${prefix}_sensor_frame">
       <sensor name="realsense_d435" type="rgbd_camera">
-        <gz_frame_id>${prefix}_optical_frame</gz_frame_id>
+        <gz_frame_id>${prefix}_sensor_frame</gz_frame_id>
         <update_rate>30</update_rate>
         <topic>${prefix}/realsense_d435</topic>
         <camera name="camera">
+          <optical_frame_id>${prefix}_optical_frame</optical_frame_id>
           <horizontal_fov>1.0472</horizontal_fov>
           <lens>
@@ -58,4 +65,11 @@
               <s>0</s>
             </intrinsics>
+            <projection>
+              <!-- same as intrinsics -->
+              <p_fx>554.25469</p_fx>
+              <p_fy>554.25469</p_fy>
+              <p_cx>320.5</p_cx>
+              <p_cy>240.5</p_cy>
+            </projection>
           </lens>
           <distortion>

Commit message: Add map to rviz config and disable IMU orientation publish

File: src/maly_woz_description/urdf/sensors/realsense_d435/realsense_d435.urdf.xacro (robot description, xacro)
@@ -17,4 +17,5 @@
       </inertial>
       <collision name="collision">
+        <origin xyz="0 0 0" rpy="0 0 ${pi / 2}"/>
         <geometry>
           <mesh filename="file://${sensor_path}/meshes/realsense.dae" />
@@ -111,4 +112,7 @@
         <visualize>true</visualize>
         <topic>${prefix}/imu</topic>
+        <imu>
+          <enable_orientation>false</enable_orientation>
+        </imu>
       </sensor>
     </gazebo>
